File: pcb/video_streamer.kicad_pcb (KiCad board)
At the start: 2 copper layers, 52 parts, among them U1 ICE40HX4K-144, U2 AT25SF041-SSHD, U3 KSZ9031RNXCA, U4 EP2C8Q208, U5 OV7670_module, U6 OV7670_module, U7 OV7670_module, U8 OV7670_module

Commit message: Cleanup files.
Parts:
- added U10: OV7670_module, Connector_PinSocket_2.54mm:PinSocket_2x09_P2.54mm_Vertical, F.Cu at (196.1, -133.3)
- added U11: OV7670_module, Connector_PinSocket_2.54mm:PinSocket_2x09_P2.54mm_Horizontal, F.Cu at (211.0, -105.7)
- added U12: OV7670_module, Connector_PinSocket_2.54mm:PinSocket_2x09_P2.54mm_Vertical, F.Cu at (196.1, -105.6)
- added U13: OV7670_module, Connector_PinSocket_2.54mm:PinSocket_2x09_P2.54mm_Horizontal, F.Cu at (257.8, -133.4)
- added U14: OV7670_module, Connector_PinSocket_2.54mm:PinSocket_2x09_P2.54mm_Vertical, F.Cu at (243.0, -133.3)
- added U15: OV7670_module, Connector_PinSocket_2.54mm:PinSocket_2x09_P2.54mm_Horizontal, F.Cu at (257.8, -105.7)
- added U16: OV7670_module, Connector_PinSocket_2.54mm:PinSocket_2x09_P2.54mm_Vertical, F.Cu at (243.0, -105.6)
- added U17: OV7670_module, Connector_PinSocket_2.54mm:PinSocket_2x09_P2.54mm_Horizontal, F.Cu at (304.7, -133.4)
- added U18: OV7670_module, Connector_PinSocket_2.54mm:PinSocket_2x09_P2.54mm_Vertical, F.Cu at (289.8, -133.3)
- added U19: OV7670_module, Connector_PinSocket_2.54mm:PinSocket_2x09_P2.54mm_Horizontal, F.Cu at (304.7, -105.7)
- added U20: OV7670_module, Connector_PinSocket_2.54mm:PinSocket_2x09_P2.54mm_Vertical, F.Cu at (289.8, -105.6)
- added U9: OV7670_module, Connector_PinSocket_2.54mm:PinSocket_2x09_P2.54mm_Horizontal, F.Cu at (211.0, -133.4)
Connections:
- U5 pad 10: /OV7670 Sensor/ov_d6 -> /OV7670 Sensor 0/ov_d6
- U5 pad 11: /OV7670 Sensor/ov_d5 -> /OV7670 Sensor 0/ov_d5
- U5 pad 12: /OV7670 Sensor/ov_d4 -> /OV7670 Sensor 0/ov_d4
- U5 pad 13: /OV7670 Sensor/ov_d3 -> /OV7670 Sensor 0/ov_d3
- U5 pad 14: /OV7670 Sensor/ov_d2 -> /OV7670 Sensor 0/ov_d2
- U5 pad 15: /OV7670 Sensor/ov_d1 -> /OV7670 Sensor 0/ov_d1
- U5 pad 16: /OV7670 Sensor/ov_d0 -> /OV7670 Sensor 0/ov_d0
- U5 pad 9: /OV7670 Sensor/ov_d7 -> /OV7670 Sensor 0/ov_d7
- U6 pad 10: /OV7670 Sensor/ov_d6 -> /OV7670 Sensor 0/ov_d6
- U6 pad 11: /OV7670 Sensor/ov_d5 -> /OV7670 Sensor 0/ov_d5
- U6 pad 12: /OV7670 Sensor/ov_d4 -> /OV7670 Sensor 0/ov_d4
- U6 pad 13: /OV7670 Sensor/ov_d3 -> /OV7670 Sensor 0/ov_d3
- U6 pad 14: /OV7670 Sensor/ov_d2 -> /OV7670 Sensor 0/ov_d2
- U6 pad 15: /OV7670 Sensor/ov_d1 -> /OV7670 Sensor 0/ov_d1
- U6 pad 16: /OV7670 Sensor/ov_d0 -> /OV7670 Sensor 0/ov_d0
- U6 pad 9: /OV7670 Sensor/ov_d7 -> /OV7670 Sensor 0/ov_d7
- U7 pad 10: /OV7670 Sensor/ov_d6 -> /OV7670 Sensor 1/ov_d6
- U7 pad 11: /OV7670 Sensor/ov_d5 -> /OV7670 Sensor 1/ov_d5
- U7 pad 12: /OV7670 Sensor/ov_d4 -> /OV7670 Sensor 1/ov_d4
- U7 pad 13: /OV7670 Sensor/ov_d3 -> /OV7670 Sensor 1/ov_d3
- U7 pad 14: /OV7670 Sensor/ov_d2 -> /OV7670 Sensor 1/ov_d2
- U7 pad 15: /OV7670 Sensor/ov_d1 -> /OV7670 Sensor 1/ov_d1
- U7 pad 16: /OV7670 Sensor/ov_d0 -> /OV7670 Sensor 1/ov_d0
- U7 pad 9: /OV7670 Sensor/ov_d7 -> /OV7670 Sensor 1/ov_d7
- U8 pad 10: /OV7670 Sensor/ov_d6 -> /OV7670 Sensor 1/ov_d6
- U8 pad 11: /OV7670 Sensor/ov_d5 -> /OV7670 Sensor 1/ov_d5
- U8 pad 12: /OV7670 Sensor/ov_d4 -> /OV7670 Sensor 1/ov_d4
- U8 pad 13: /OV7670 Sensor/ov_d3 -> /OV7670 Sensor 1/ov_d3
- U8 pad 14: /OV7670 Sensor/ov_d2 -> /OV7670 Sensor 1/ov_d2
- U8 pad 15: /OV7670 Sensor/ov_d1 -> /OV7670 Sensor 1/ov_d1
- U8 pad 16: /OV7670 Sensor/ov_d0 -> /OV7670 Sensor 1/ov_d0
- U8 pad 9: /OV7670 Sensor/ov_d7 -> /OV7670 Sensor 1/ov_d7
Routing:
- net /OV7670 Sensor/ov_d0: track 10.4 -> 0.00 mm
- net /OV7670 Sensor 0/ov_d0: track 0.00 -> 10.4 mm
- net /OV7670 Sensor/ov_d6: track 10.4 -> 0.00 mm
- net /OV7670 Sensor/ov_d4: track 10.4 -> 0.00 mm
- net /OV7670 Sensor 0/ov_d6: track 0.00 -> 10.4 mm
- net /OV7670 Sensor 0/ov_d4: track 0.00 -> 10.4 mm
- net /OV7670 Sensor/ov_d7: track 10.4 -> 0.00 mm
- net /OV7670 Sensor/ov_d5: track 10.4 -> 0.00 mm
- net /OV7670 Sensor 0/ov_d7: track 0.00 -> 10.4 mm
- net /OV7670 Sensor 0/ov_d5: track 0.00 -> 10.4 mm
- net /OV7670 Sensor/ov_d3: track 10.4 -> 0.00 mm
- net /OV7670 Sensor/ov_d1: track 10.4 -> 0.00 mm
- net /OV7670 Sensor 0/ov_d3: track 0.00 -> 10.4 mm
- net /OV7670 Sensor 0/ov_d1: track 0.00 -> 10.4 mm

Commit message: OV flat footprint
Parts:
- U11, U13, U15, U17, U19, U5, U7, U9: footprint Connector_PinSocket_2.54mm:PinSocket_2x09_P2.54mm_Horizontal -> OV7670_Module:OV7670_Flat
- moved U17 320.7 mm to (78.0, 93.5), turned to 180 degrees
- moved U13 306.3 mm to (128.0, 144.0), turned to 270 degrees
- moved U15 287.1 mm to (92.5, 129.0), turned to 225 degrees
- moved U19 267.6 mm to (93.0, 57.9), turned to 135 degrees
- moved U11 240.0 mm to (163.6, 129.5), turned to 315 degrees
- moved U9 229.6 mm to (178.6, 94.0)
- moved U10 223.8 mm to (158.8, 87.4)
- moved U6 168.7 mm to (104.9, -18.5), turned to 270 degrees
- moved U4 167.9 mm to (128.3, 93.7)
- moved U5 145.2 mm to (128.5, 43.4), turned to 90 degrees
- moved U8 139.8 mm to (124.5, 66.8), turned to 90 degrees
- moved U7 111.0 mm to (164.1, 58.4), turned to 45 degrees
Connections:
- U11 pad 10: /OV7670 Sensor 2/ov_d6 -> /OV7670 Sensor 3/ov_d6
- U11 pad 11: /OV7670 Sensor 2/ov_d5 -> /OV7670 Sensor 3/ov_d5
- U11 pad 12: /OV7670 Sensor 2/ov_d4 -> /OV7670 Sensor 3/ov_d4
- U11 pad 13: /OV7670 Sensor 2/ov_d3 -> /OV7670 Sensor 3/ov_d3
- U11 pad 14: /OV7670 Sensor 2/ov_d2 -> /OV7670 Sensor 3/ov_d2
- U11 pad 15: /OV7670 Sensor 2/ov_d1 -> /OV7670 Sensor 3/ov_d1
- U11 pad 16: /OV7670 Sensor 2/ov_d0 -> /OV7670 Sensor 3/ov_d0
- U11 pad 3: /ov2_soic -> /ov3_soic
- U11 pad 5: /ov2_vsync -> /ov3_vsync
- U11 pad 6: /ov2_href -> /ov3_href
- U11 pad 7: /ov2_pclk -> /ov3_pclk
- U11 pad 9: /OV7670 Sensor 2/ov_d7 -> /OV7670 Sensor 3/ov_d7
- U12 pad 10: /OV7670 Sensor 2/ov_d6 -> /OV7670 Sensor 3/ov_d6
- U12 pad 11: /OV7670 Sensor 2/ov_d5 -> /OV7670 Sensor 3/ov_d5
- U12 pad 12: /OV7670 Sensor 2/ov_d4 -> /OV7670 Sensor 3/ov_d4
- U12 pad 13: /OV7670 Sensor 2/ov_d3 -> /OV7670 Sensor 3/ov_d3
- U12 pad 14: /OV7670 Sensor 2/ov_d2 -> /OV7670 Sensor 3/ov_d2
- U12 pad 15: /OV7670 Sensor 2/ov_d1 -> /OV7670 Sensor 3/ov_d1
- U12 pad 16: /OV7670 Sensor 2/ov_d0 -> /OV7670 Sensor 3/ov_d0
- U12 pad 3: /ov2_soic -> /ov3_soic
- U12 pad 5: /ov2_vsync -> /ov3_vsync
- U12 pad 6: /ov2_href -> /ov3_href
- U12 pad 7: /ov2_pclk -> /ov3_pclk
- U12 pad 9: /OV7670 Sensor 2/ov_d7 -> /OV7670 Sensor 3/ov_d7
- U13 pad 10: /OV7670 Sensor 0/ov_d6 -> /OV7670 Sensor 4/ov_d6
- U13 pad 11: /OV7670 Sensor 0/ov_d5 -> /OV7670 Sensor 4/ov_d5
- U13 pad 12: /OV7670 Sensor 0/ov_d4 -> /OV7670 Sensor 4/ov_d4
- U13 pad 13: /OV7670 Sensor 0/ov_d3 -> /OV7670 Sensor 4/ov_d3
- U13 pad 14: /OV7670 Sensor 0/ov_d2 -> /OV7670 Sensor 4/ov_d2
- U13 pad 15: /OV7670 Sensor 0/ov_d1 -> /OV7670 Sensor 4/ov_d1
- U13 pad 16: /OV7670 Sensor 0/ov_d0 -> /OV7670 Sensor 4/ov_d0
- U13 pad 3: /ov0_soic -> /ov4_soic
- U13 pad 5: /ov0_vsync -> /ov4_vsync
- U13 pad 6: /ov0_href -> /ov4_href
- U13 pad 7: /ov0_pclk -> /ov4_pclk
- U13 pad 9: /OV7670 Sensor 0/ov_d7 -> /OV7670 Sensor 4/ov_d7
- U14 pad 10: /OV7670 Sensor 0/ov_d6 -> /OV7670 Sensor 4/ov_d6
- U14 pad 11: /OV7670 Sensor 0/ov_d5 -> /OV7670 Sensor 4/ov_d5
- U14 pad 12: /OV7670 Sensor 0/ov_d4 -> /OV7670 Sensor 4/ov_d4
- U14 pad 13: /OV7670 Sensor 0/ov_d3 -> /OV7670 Sensor 4/ov_d3
- U14 pad 14: /OV7670 Sensor 0/ov_d2 -> /OV7670 Sensor 4/ov_d2
- U14 pad 15: /OV7670 Sensor 0/ov_d1 -> /OV7670 Sensor 4/ov_d1
- U14 pad 16: /OV7670 Sensor 0/ov_d0 -> /OV7670 Sensor 4/ov_d0
- U14 pad 3: /ov0_soic -> /ov4_soic
- U14 pad 5: /ov0_vsync -> /ov4_vsync
- U14 pad 6: /ov0_href -> /ov4_href
- U14 pad 7: /ov0_pclk -> /ov4_pclk
- U14 pad 9: /OV7670 Sensor 0/ov_d7 -> /OV7670 Sensor 4/ov_d7
- U15 pad 10: /OV7670 Sensor 1/ov_d6 -> /OV7670 Sensor 5/ov_d6
- U15 pad 11: /OV7670 Sensor 1/ov_d5 -> /OV7670 Sensor 5/ov_d5
- U15 pad 12: /OV7670 Sensor 1/ov_d4 -> /OV7670 Sensor 5/ov_d4
- U15 pad 13: /OV7670 Sensor 1/ov_d3 -> /OV7670 Sensor 5/ov_d3
- U15 pad 14: /OV7670 Sensor 1/ov_d2 -> /OV7670 Sensor 5/ov_d2
- U15 pad 15: /OV7670 Sensor 1/ov_d1 -> /OV7670 Sensor 5/ov_d1
- U15 pad 16: /OV7670 Sensor 1/ov_d0 -> /OV7670 Sensor 5/ov_d0
- U15 pad 3: /ov1_soic -> /ov5_soic
- U15 pad 5: /ov1_vsync -> /ov5_vsync
- U15 pad 6: /ov1_href -> /ov5_href
- U15 pad 7: /ov1_pclk -> /ov5_pclk
- U15 pad 9: /OV7670 Sensor 1/ov_d7 -> /OV7670 Sensor 5/ov_d7
- U16 pad 10: /OV7670 Sensor 1/ov_d6 -> /OV7670 Sensor 5/ov_d6
- U16 pad 11: /OV7670 Sensor 1/ov_d5 -> /OV7670 Sensor 5/ov_d5
- U16 pad 12: /OV7670 Sensor 1/ov_d4 -> /OV7670 Sensor 5/ov_d4
- U16 pad 13: /OV7670 Sensor 1/ov_d3 -> /OV7670 Sensor 5/ov_d3
- U16 pad 14: /OV7670 Sensor 1/ov_d2 -> /OV7670 Sensor 5/ov_d2
- U16 pad 15: /OV7670 Sensor 1/ov_d1 -> /OV7670 Sensor 5/ov_d1
- U16 pad 16: /OV7670 Sensor 1/ov_d0 -> /OV7670 Sensor 5/ov_d0
- U16 pad 3: /ov1_soic -> /ov5_soic
- U16 pad 5: /ov1_vsync -> /ov5_vsync
- U16 pad 6: /ov1_href -> /ov5_href
- U16 pad 7: /ov1_pclk -> /ov5_pclk
- U16 pad 9: /OV7670 Sensor 1/ov_d7 -> /OV7670 Sensor 5/ov_d7
- U17 pad 10: /OV7670 Sensor 2/ov_d6 -> /OV7670 Sensor 6/ov_d6
- U17 pad 11: /OV7670 Sensor 2/ov_d5 -> /OV7670 Sensor 6/ov_d5
- U17 pad 12: /OV7670 Sensor 2/ov_d4 -> /OV7670 Sensor 6/ov_d4
- U17 pad 13: /OV7670 Sensor 2/ov_d3 -> /OV7670 Sensor 6/ov_d3
- U17 pad 14: /OV7670 Sensor 2/ov_d2 -> /OV7670 Sensor 6/ov_d2
- U17 pad 15: /OV7670 Sensor 2/ov_d1 -> /OV7670 Sensor 6/ov_d1
- U17 pad 16: /OV7670 Sensor 2/ov_d0 -> /OV7670 Sensor 6/ov_d0
- U17 pad 3: /ov2_soic -> /ov6_soic
- U17 pad 5: /ov2_vsync -> /ov6_vsync
- U17 pad 6: /ov2_href -> /ov6_href
- U17 pad 7: /ov2_pclk -> /ov6_pclk
- U17 pad 9: /OV7670 Sensor 2/ov_d7 -> /OV7670 Sensor 6/ov_d7
- U18 pad 10: /OV7670 Sensor 2/ov_d6 -> /OV7670 Sensor 6/ov_d6
- U18 pad 11: /OV7670 Sensor 2/ov_d5 -> /OV7670 Sensor 6/ov_d5
- U18 pad 12: /OV7670 Sensor 2/ov_d4 -> /OV7670 Sensor 6/ov_d4
- U18 pad 13: /OV7670 Sensor 2/ov_d3 -> /OV7670 Sensor 6/ov_d3
- U18 pad 14: /OV7670 Sensor 2/ov_d2 -> /OV7670 Sensor 6/ov_d2
- U18 pad 15: /OV7670 Sensor 2/ov_d1 -> /OV7670 Sensor 6/ov_d1
- U18 pad 16: /OV7670 Sensor 2/ov_d0 -> /OV7670 Sensor 6/ov_d0
- U18 pad 3: /ov2_soic -> /ov6_soic
- U18 pad 5: /ov2_vsync -> /ov6_vsync
- U18 pad 6: /ov2_href -> /ov6_href
- U18 pad 7: /ov2_pclk -> /ov6_pclk
- U18 pad 9: /OV7670 Sensor 2/ov_d7 -> /OV7670 Sensor 6/ov_d7
- U19 pad 10: /OV7670 Sensor 2/ov_d6 -> /OV7670 Sensor 7/ov_d6
- U19 pad 11: /OV7670 Sensor 2/ov_d5 -> /OV7670 Sensor 7/ov_d5
- U19 pad 12: /OV7670 Sensor 2/ov_d4 -> /OV7670 Sensor 7/ov_d4
- U19 pad 13: /OV7670 Sensor 2/ov_d3 -> /OV7670 Sensor 7/ov_d3
- U19 pad 14: /OV7670 Sensor 2/ov_d2 -> /OV7670 Sensor 7/ov_d2
- U19 pad 15: /OV7670 Sensor 2/ov_d1 -> /OV7670 Sensor 7/ov_d1
- U19 pad 16: /OV7670 Sensor 2/ov_d0 -> /OV7670 Sensor 7/ov_d0
- U19 pad 3: /ov2_soic -> /ov7_soic
- U19 pad 5: /ov2_vsync -> /ov7_vsync
- U19 pad 6: /ov2_href -> /ov7_href
- U19 pad 7: /ov2_pclk -> /ov7_pclk
- U19 pad 9: /OV7670 Sensor 2/ov_d7 -> /OV7670 Sensor 7/ov_d7
- U20 pad 10: /OV7670 Sensor 2/ov_d6 -> /OV7670 Sensor 7/ov_d6
- U20 pad 11: /OV7670 Sensor 2/ov_d5 -> /OV7670 Sensor 7/ov_d5
- U20 pad 12: /OV7670 Sensor 2/ov_d4 -> /OV7670 Sensor 7/ov_d4
- U20 pad 13: /OV7670 Sensor 2/ov_d3 -> /OV7670 Sensor 7/ov_d3
- U20 pad 14: /OV7670 Sensor 2/ov_d2 -> /OV7670 Sensor 7/ov_d2
- U20 pad 15: /OV7670 Sensor 2/ov_d1 -> /OV7670 Sensor 7/ov_d1
- U20 pad 16: /OV7670 Sensor 2/ov_d0 -> /OV7670 Sensor 7/ov_d0
- U20 pad 3: /ov2_soic -> /ov7_soic
- U20 pad 5: /ov2_vsync -> /ov7_vsync
- U20 pad 6: /ov2_href -> /ov7_href
- U20 pad 7: /ov2_pclk -> /ov7_pclk
- U20 pad 9: /OV7670 Sensor 2/ov_d7 -> /OV7670 Sensor 7/ov_d7
Routing:
- net /OV7670 Sensor/ov_d2: track 61.6 -> 0.00 mm
- net /OV7670 Sensor 1/ov_d2: track 0.00 -> 49.6 mm
- net +3V3: track 11.0 -> 0.00 mm
- net /ov_xclk: track 10.4 -> 0.00 mm
- net /ov_soid: track 10.4 -> 0.00 mm
- net /ov0_href: track 10.4 -> 0.00 mm
- net /OV7670 Sensor 0/ov_d0: track 10.4 -> 0.00 mm
- net /ov_pwdn: track 10.4 -> 0.00 mm
- net /OV7670 Sensor 0/ov_d6: track 10.4 -> 0.00 mm
- net /OV7670 Sensor 0/ov_d4: track 10.4 -> 0.00 mm
- net GNDD: track 155.9 -> 145.5 mm
- net /ov0_soic: track 10.4 -> 0.00 mm
- net /ov_reset: track 10.4 -> 0.00 mm
- net /ov0_vsync: track 10.4 -> 0.00 mm
- net /OV7670 Sensor 0/ov_d7: track 10.4 -> 0.00 mm
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
Commit message: Cameras angled 22.5.
Parts:
- U10, U12, U14, U16, U18, U20, U6, U8: footprint Connector_PinSocket_2.54mm:PinSocket_2x09_P2.54mm_Vertical -> OV7670_Module:OV7670_Vertical
- moved U14 332.7 mm to (37.9, 128.6), turned to 290 degrees
- moved U18 266.0 mm to (81.4, 32.0), turned to 315 degrees
- moved U16 242.0 mm to (61.4, 54.4), turned to 337.5 degrees
- moved U20 219.8 mm to (108.6, 18.7), turned to 292.5 degrees
- moved U4 214.1 mm to (-74.7, 161.7)
- moved U12 178.9 mm to (202.9, 73.2), turned to 202.5 degrees
- moved U19 68.0 mm to (128.3, 116.1), turned to 270 degrees
- moved U8 58.3 mm to (166.6, 26.5), turned to 247.5 degrees
- moved U10 51.3 mm to (189.5, 46.3), turned to 225 degrees
- moved U6 48.8 mm to (138.4, 16.9)
- moved U7 37.9 mm to (128.3, 70.9), turned to 270 degrees
- moved U9 23.2 mm to (180.3, 70.9), turned to 270 degrees
- moved U17 22.7 mm to (76.3, 70.9), turned to 270 degrees
- moved U11 21.4 mm to (180.3, 116.1), turned to 270 degrees
- moved U15 20.7 mm to (76.3, 116.1), turned to 270 degrees
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Routing:
- net /ov2_vsync: track 0.00 -> 12.4 mm
- net /OV7670 Sensor 1/ov_d2: track 49.6 -> 37.1 mm

Commit message: Remove one flat sensor site.
Parts:
- removed U13, U5: OV7670_module, OV7670_Module:OV7670_Flat
- removed U14: OV7670_module, OV7670_Module:OV7670_Vertical
- moved U4 236.5 mm to (128.3, 40.4)
- moved U3 167.4 mm to (128.3, 138.2)
Routing:
- net GNDD: track 145.5 -> 0.00 mm
- net /OV7670 Sensor 1/ov_d2: track 37.1 -> 0.00 mm
- net /ICE40/spi_sdi: track 16.6 -> 0.55 mm, vias 2 -> 0
- net /ICE40/spi_sck: track 16.7 -> 0.84 mm, vias 2 -> 0
- net /ov2_vsync: track 12.4 -> 0.00 mm
- net /ICE40/spi_ss: track 7.62 -> 0.00 mm
- net /ICE40/spi_sdo: track 8.02 -> 1.00 mm
